File: Phi Schematics/Phi.sch (EAGLE design)
At the start: 10 parts

Commit message: phi schematics
Parts:
- removed JOINT_POS, MOT_HIP, MOT_KNEE: (no value), pinhead:PINHD-1X2
- removed JP1: (no value), pinhead:PINHD-1X3
- removed R_HIP, R_KNEE: (no value), pot:TRIM_EU-B25P
- removed U$2: QIK_2S9V1, Misc-Phi-Comp:QIK_2S9V1
- removed U$3, U$4: DC-MOTOR, Misc-Phi-Comp:DC-MOTOR
- added BAT1: (no value), special:BATTERY
- added C1, C2: (no value), capacitor-wima:C2,5-3
- added JOINT_POS1, MOT_HIP1, MOT_KNEE1: (no value), pinhead:PINHD-1X2
- added JP2: (no value), pinhead:PINHD-1X3
- added POT, POT1, R_HIP1, R_KNEE1, R_RFH, R_RFH1, R_RFH2: (no value), pot:TRIM_EU-B25P
- added R1: (no value), rcl:R-EU_0204/2V
- added U$5: QIK_2S9V1, Misc-Phi-Comp:QIK_2S9V1
- added U$6, U$7: DC-MOTOR, Misc-Phi-Comp:DC-MOTOR
Connections:
- removed net N$10: MOT_HIP.1, U$2.M0+, U$3.M+
- removed net N$7: JOINT_POS.1, R_HIP.S
- removed net N$8: JOINT_POS.2, R_KNEE.S
- removed net TX/RX: JP1.1, U$1.8-TX, U$2.RX
- new net +3V1: JP2.2, U$5.LOG_VCC
- new net N$1: U$1.24-SPI-CE0-N
- new net N$12: JOINT_POS1.2, R_KNEE1.S
- new net N$13: MOT_KNEE1.2, U$5.M1-, U$7.M-
- new net N$14: MOT_HIP1.1, U$5.M0+, U$6.M+
- new net N$15: JOINT_POS1.1, R_HIP1.S
- new net N$2: MOT_HIP1.2, U$5.M0-, U$6.M-
- new net N$6: C2.2
- new net N$9: MOT_KNEE1.1, U$5.M1+, U$7.M+
- new net RFH: R_RFH2.S
- new net RFH1: C1.1, POT.S
- new net RFH2: C2.1, POT1.S, R1.2
- new net RFK: R_RFH1.S
- new net RFT: R_RFH.S
- new net SPI-CLK: U$1.23-SPI-SCLK
- new net SPI-MISO: U$1.21-SPI-MISO
- new net SPI-MOSI: U$1.19-SPI-MOSI
- new net TX/RX1: JP2.1, U$5.RX
- new net UART-TX: U$1.8-TX
- net +3V3: no longer JP1.2, U$2.LOG_VCC
- net +5V: now also BAT1.+, JP2.3, POT.E, POT1.E, R_HIP1.E, R_KNEE1.E, R_RFH.E, R_RFH1.E, R_RFH2.E, U$5.VMOT; no longer JP1.3, R_HIP.E, R_KNEE.E, U$2.VMOT
- net GND: now also BAT1.-, POT.A, R1.1, R_HIP1.A, R_KNEE1.A, R_RFH.A, R_RFH1.A, R_RFH2.A, U$5.LOG_GND, U$5.MOT_GND; no longer U$1.6-GND, U$2.LOG_GND, U$2.MOT_GND
- net N$3: now also U$1.26-SPI-CE1-N; no longer MOT_HIP.2, U$2.M0-, U$3.M-
- net N$4: now also U$1.6-GND; no longer MOT_KNEE.2, U$2.M1-, U$4.M-
- net N$5: now also C1.2; no longer MOT_KNEE.1, U$2.M1+, U$4.M+
